Commit message: 统一kinect2的描述文件

File: turtlebot2i_description/urdf/sensors/kinect2.urdf.xacro (robot description, xacro)
@@ -9,7 +9,7 @@
       <origin xyz="-0.119 0.125 0.306" rpy="${cam_or} ${cam_op} ${cam_oy}"/>
       <parent link="${parent}"/>
-      <child link="camera_link" />
+      <child link="kinect2_model_link" />
     </joint>
-    <link name="camera_link">
+    <link name="kinect2_model_link">
       <visual>
        <origin xyz="0 0 0" rpy="-0.11757 0 -1.5707963"/>
@@ -36,10 +36,10 @@
     </link>
     <joint name="camera_rgb_joint" type="fixed">
-      <origin xyz="0.080 -0.2198 0.0317" rpy="${cam_or} ${cam_op} ${cam_oy}"/>
-      <parent link="camera_link"/>
+      <origin xyz="0.080 -0.2198 0.0317" rpy="0 0 0"/>
+      <parent link="kinect2_model_link"/>
       <child link="camera_rgb_frame" />
     </joint>
     <link name="camera_rgb_frame"/>
-    <joint name="kinect2_model_joint" type="fixed">
+    <joint name="camera_rgb_optical_joint" type="fixed">
       <origin xyz="0.0 0.0 0.0" rpy="-1.570796327 0.0 -1.570796327"/>
       <parent link="camera_rgb_frame"/>
@@ -50,30 +50,30 @@
          files. However, for Gazebo simulation we need them, so we add them here.
          (Hence, don't publish them additionally!) -->
-	<joint name="camera_depth_joint" type="fixed">
-	  <origin xyz="0 0.05 0" rpy="0 0 0" />
-	  <parent link="camera_rgb_frame" />
-	  <child link="camera_depth_frame" />
-	</joint>
-	<link name="camera_depth_frame"/>
-	<joint name="camera_ir_joint" type="fixed">
-	  <origin xyz="0 0.05 0" rpy="0 0 0" />
-	  <parent link="camera_rgb_frame" />
-	  <child link="camera_ir_frame" />
-	</joint>
-	<link name="camera_ir_frame"/>
-	<joint name="camera_depth_optical_joint" type="fixed">
-	  <origin xyz="0 0 0" rpy="-1.570796327 0.0 -1.570796327" />
-	  <parent link="camera_depth_frame" />
-	  <child link="camera_depth_optical_frame" />
-	</joint>
-	<link name="camera_ir_optical_frame"/>
-	<joint name="camera_ir_optical_joint" type="fixed">
-	  <origin xyz="0 0 0" rpy="-1.570796327 0.0 -1.570796327" />
-	  <parent link="camera_ir_frame" />
-	  <child link="camera_ir_optical_frame" />
-	</joint>
-	<link name="camera_depth_optical_frame"/>
-	<!-- Kinect sensor for simulation -->
-	<turtlebot_sim_3dsensor/>
+	  <joint name="camera_depth_joint" type="fixed">
+	    <origin xyz="0 0.05 0" rpy="0 0 0" />
+	    <parent link="camera_rgb_frame" />
+	    <child link="camera_depth_frame" />
+	  </joint>
+	  <link name="camera_depth_frame"/>
+	  <joint name="camera_depth_optical_joint" type="fixed">
+	    <origin xyz="0 0 0" rpy="${-M_PI/2} 0.0 ${-M_PI/2}" />
+	    <parent link="camera_depth_frame" />
+	    <child link="camera_depth_optical_frame" />
+	  </joint>
+	  <link name="camera_depth_optical_frame"/>
+	  <joint name="camera_ir_joint" type="fixed">
+	    <origin xyz="0 0.05 0" rpy="0 0 0" />
+	    <parent link="camera_rgb_frame" />
+	    <child link="camera_ir_frame" />
+	  </joint>
+    <link name="camera_ir_frame"/>
+    <joint name="camera_ir_optical_joint" type="fixed">
+	    <origin xyz="0 0 0" rpy="-1.570796327 0.0 -1.570796327" />
+	    <parent link="camera_ir_frame" />
+	    <child link="camera_ir_optical_frame" />
+	  </joint>
+    <link name="camera_ir_optical_frame"/>
+	  <!-- Kinect sensor for simulation -->
+	  <turtlebot_sim_3dsensor/>
   </xacro:macro>
 </robot>

Commit message: 修改了kinect2的皮肤路径

File: turtlebot2i_description/urdf/sensors/kinect2.urdf.xacro (robot description, xacro)
@@ -15,5 +15,5 @@
        <origin xyz="0 0 0" rpy="-0.11757 0 -1.5707963"/>
         <geometry>
-         <mesh filename="package://turtlebot_description/meshes/sensors/kinect2.stl" scale="0.001 0.001 0.001"/>
+         <mesh filename="package://turtlebot2i_description/meshes/sensors/kinect2.stl" scale="0.001 0.001 0.001"/>
         </geometry>
         <material name="black">

Commit message: 修改kinect2的高度

File: turtlebot2i_description/urdf/sensors/kinect2.urdf.xacro (robot description, xacro)
@@ -7,5 +7,5 @@
   <xacro:macro name="sensor_kinect2" params="parent">
     <joint name="camera_mount_joint" type="fixed">
-      <origin xyz="-0.119 0.125 0.306" rpy="${cam_or} ${cam_op} ${cam_oy}"/>
+      <origin xyz="-0.119 0.125 0.256" rpy="${cam_or} ${cam_op} ${cam_oy}"/>
       <parent link="${parent}"/>
       <child link="kinect2_model_link" />
