Commit message: 微调sr300的姿态以适应机器人

File: turtlebot2i_description/urdf/sensors/sr300.urdf.xacro (robot description, xacro)
@@ -4,6 +4,8 @@
   <xacro:include filename="$(find turtlebot2i_description)/urdf/turtlebot_properties.urdf.xacro"/>
   <!-- Intel SR300 parameters -->
-  <xacro:property name="sr300_cam_offset_px" value="0.138" />
-  <xacro:property name="sr300_cam_offset_py" value="0.0" />
+  <!-- <xacro:property name="sr300_cam_offset_px" value="0.138" /> -->
+  <xacro:property name="sr300_cam_offset_px" value="0.165" />
+  <!-- <xacro:property name="sr300_cam_offset_py" value="0.0" /> -->
+  <xacro:property name="sr300_cam_offset_py" value="-0.005" />
   <xacro:property name="sr300_cam_offset_pz" value="0.444" />
   <xacro:property name="sr300_cam_rgb_px" value="0.0"/>
